File: GeekyPCB/GeekyPCB.kicad_pcb (KiCad board)
At the start: 2 copper layers, 54.5 x 67.5 mm, 36 parts, among them J1 USB_C_Receptacle_USB2.0_14P, J2 DEBUG, J3 Conn_01x20, J4 Conn_01x20, SW1 SW_Push, SW2 BOOTSEL, U1 RP2040, U2 AMS1117-3.3, U3 W25Q128JVS, Y1 12MHz

Commit message: elo
Parts:
- renumbered REF** to REF67, REF** to REF68
Routing:
- net +3.3V: track 293.4 -> 292.2 mm
- net QSPI_SS: track 129.5 -> 129.0 mm
- added copper zone on F.Cu, net GND

Commit message: final
Routing:
- net +5V: track 139.2 -> 132.7 mm
- net +3.3V: track 292.2 -> 288.7 mm
